File: PCB/rf-link/rf-link.kicad_pcb (KiCad board)
At the start: 2 copper layers, 55 x 19 mm, 43 parts, among them J1 USB_A, J2 USART, J3 ANT, J4 ANT, P1 ICT-Point, P2 ICT-Point, P3 ICT-Point, P4 ICT-Point, P5 ICT-Point, P6 ICT-Point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

Commit message: add stuff
Parts:
- removed REF** (x2): MountingHole_2.2mm_M2, MountingHole:MountingHole_2.2mm_M2
- J1: footprint Connector_USB:USB_A_CONNFLY_DS1095-WNR0 -> Connector_USB:USB_Micro-B_Wuerth_629105150521
- P1, P2, P3, P4, P5, P6, P7, P8: footprint TestPoint:TestPoint_Pad_D1.5mm -> TestPoint:TestPoint_Pad_D1.0mm
- moved J1 3.93 mm to (79.8, 52.5)
- moved P8 3.34 mm to (96.3, 50.8)
- moved P6 2.74 mm to (94.8, 50.8)
- moved P2 2.43 mm to (97.8, 50.8)
- moved P7 2.41 mm to (96.3, 49.3)
- moved P5 1.78 mm to (94.8, 49.3)
- moved P3 1.04 mm to (93.3, 49.3)
- moved R1 0.47 mm to (84.6, 53.0)
- moved D1 0.31 mm to (85.4, 49.3)
- moved D2 0.31 mm to (85.4, 46.7)
- moved R2 0.31 mm to (84.6, 51.4)
- moved P4 0.05 mm to (93.3, 50.8)
Connections:
- J1 pad 4: GND -> (no net)
Routing:
- net Net-(P6-Pad1): track 1.40 -> 4.08 mm
- net Net-(P2-Pad1): track 3.12 -> 5.70 mm
- net Net-(P7-Pad1): track 4.68 -> 2.34 mm
- net Net-(P5-Pad1): track 4.27 -> 2.37 mm
- net Net-(P8-Pad1): track 2.39 -> 4.11 mm
- net VBUS: track 13.8 -> 15.4 mm
- net +5V: track 37.1 -> 38.3 mm, vias 2 -> 0
- net Net-(P3-Pad1): track 1.34 -> 2.40 mm
- net /D-: track 4.89 -> 3.98 mm
- net /Vsup: track 8.19 -> 9.10 mm
- net /SS: track 31.4 -> 32.1 mm
- net /D+: track 4.87 -> 4.27 mm

Commit message: Work on the rf-link usb module
Parts:
- added J5: AVR-ISP-6, Connector:Tag-Connect_TC2030-IDC-NL_2x03_P1.27mm_Vertical, F.Cu at (85.4, 57.4)
- added JP2: HWB, Jumper:SolderJumper-2_P1.3mm_Open_RoundedPad1.0x1.5mm, F.Cu at (105.2, 46.1)
- added P9: ICT-Point, TestPoint:TestPoint_Pad_D1.0mm, F.Cu at (95.6, 60.7)
- added R7: 10k, Resistor_SMD:R_0603_1608Metric, F.Cu at (103.1, 46.3)
- added REF**: MountingHole_2.2mm_M2, MountingHole:MountingHole_2.2mm_M2, F.Cu at (129.0, 44.0)
- added REF**: MountingHole_2.2mm_M2, MountingHole:MountingHole_2.2mm_M2, F.Cu at (129.0, 60.0)
- added REF**: MountingHole_2.2mm_M2, MountingHole:MountingHole_2.2mm_M2, F.Cu at (78.0, 60.0)
- added REF**: MountingHole_2.2mm_M2, MountingHole:MountingHole_2.2mm_M2, F.Cu at (78.0, 44.0)
- C6, SW1: moved to B.Cu
- J1: footprint Connector_USB:USB_Micro-B_Wuerth_629105150521 -> SilentWorks:USB_Micro-B_Futheda
- J4: footprint Connector_Coaxial:SMA_Molex_73251-2120_EdgeMount_Horizontal -> Connector_Coaxial:U.FL_Hirose_U.FL-R-SMT-1_Vertical
- P2: moved to F.Cu
- moved P2 8.23 mm to (104.9, 55.1)
- moved C6 7.25 mm to (90.6, 59.3)
- moved D3 2.97 mm to (109.5, 46.8)
- moved D4 2.97 mm to (107.4, 46.8)
- moved R4 2.97 mm to (109.5, 50.3)
- moved R5 2.97 mm to (107.4, 50.3)
- moved J1 2.29 mm to (77.5, 52.0)
- moved J3 2.17 mm to (125.8, 49.5)
- moved J4 1.44 mm to (127.5, 52.5), turned to 270 degrees
- moved P1 0.82 mm to (97.1, 60.7)
- moved SW1 0.76 mm to (85.5, 57.4), turned to 180 degrees
- moved R6 0.07 mm to (103.1, 49.3)
Connections:
- U2 pad 18: (no net) -> Net-(P9-Pad1)
- U2 pad 33: +3V3 -> Net-(JP2-Pad1)
Routing:
- net +3V3: track 79.4 -> 89.6 mm, vias 3 -> 7
- net /DIO4: track 15.2 -> 5.45 mm
- net /SCK: track 34.8 -> 44.0 mm
- net /MISO: track 34.2 -> 41.7 mm, vias 1 -> 3
- net +5V: track 38.3 -> 45.6 mm, vias 0 -> 2
- net Net-(JP2-Pad1): track 0.00 -> 5.97 mm
- net /MOSI: track 36.3 -> 39.8 mm
- net /~RST: track 10.9 -> 14.2 mm, vias 0 -> 2
- net Net-(P9-Pad1): track 0.00 -> 2.38 mm
- net /~RFM_RST: track 21.5 -> 23.8 mm
- net /SS: track 32.1 -> 29.8 mm
- net /ANT: track 9.54 -> 7.39 mm
- net /LED_RED: track 10.3 -> 12.2 mm
- net /USB_D-: track 2.36 -> 4.15 mm
- net /USB_D+: track 2.39 -> 4.15 mm
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Other:
- board size 55 x 19 mm -> 55 x 20 mm
